Commit message: Automated update by GitHub Action

File: urdf/robot.urdf (robot description, URDF)
Before this commit: robot robot, 18 links, 17 joints
Links:
- removed link motor_holder
- added link base_link, mass 1.06123; collision mesh filename=package://catbot_leg_description/meshes/motor_holder.stl; collision mesh filename=package://catbot_leg_description/meshes/part_1.stl
Joints:
- joint a: parent motor_holder -> base_link
- joint imu_link_frame: parent motor_holder -> base_link
- joint l: parent motor_holder -> base_link
- joint yaw: parent motor_holder -> base_link

Commit message: Automated update by GitHub Action

File: urdf/robot.urdf (robot description, URDF)
Before this commit: robot robot, 24 links, 23 joints
Joints:
- joint BR_leg1_1 (1) (1): origin xyz=0 5.55112e-17 0.029 rpy=3.14159 1.11382e-16 -1.20167 -> xyz=1.38778e-17 3.46945e-17 0.029 rpy=3.14159 1.11382e-16 -1.20167
- joint BR_leg_cyl_0_1 (1) (1): origin xyz=2.77556e-17 -0.166278 0 rpy=3.14159 3.7907e-32 1.13039e-17 -> xyz=-1.38778e-17 -0.166278 0 rpy=3.14159 3.7907e-32 1.13039e-17
- joint BR_leg_cyl_1_1 (1) (1): origin xyz=2.77556e-17 -0.207 -1.11022e-16 rpy=-3.14159 -1.4511e-31 -6.07804e-18 -> xyz=1.38778e-17 -0.207 0 rpy=-3.14159 -1.4511e-31 -6.07804e-18
- joint a: origin xyz=0.6808 -0.0642675 0.432956 rpy=1.5708 -1.25664 1.5708 -> xyz=-0.005 -0.0545 -0.0175 rpy=1.5708 -1.25664 1.5708
- joint base_link_motor_holder_fixed: origin xyz=0.6858 -0.0097675 0.450456 rpy=-3.14159 -3.30424e-16 1.5708 -> xyz=0 0 0 rpy=3.14159 2.48154e-24 1.5708
- joint base_link_part_1_2_fixed: origin xyz=0.6573 -0.0642675 0.432956 rpy=3.14159 0.464323 -1.5708 -> xyz=-0.0285 -0.0545 -0.0175 rpy=3.14159 0.464323 -1.5708
- joint base_link_part_1_3_fixed: origin xyz=0.6733 0.0647675 0.432956 rpy=1.16838e-15 -1.91646e-16 1.5708 -> xyz=-0.0125 0.074535 -0.0175 rpy=1.16838e-15 -1.91646e-16 1.5708
- joint base_link_part_1_4_fixed: origin xyz=0.6573 0.0647675 0.432956 rpy=3.14159 0.464323 -1.5708 -> xyz=-0.0285 0.074535 -0.0175 rpy=3.14159 0.464323 -1.5708
- joint base_link_part_1_fixed: origin xyz=0.6733 -0.0642675 0.432956 rpy=1.16838e-15 -1.91646e-16 1.5708 -> xyz=-0.0125 -0.0545 -0.0175 rpy=1.16838e-15 -1.91646e-16 1.5708
- joint base_link_t_slot_frame_fixed: origin xyz=0.6958 0.0005 0.946156 rpy=-3.14159 -3.30424e-16 1.5708 -> xyz=0.01 0.0102675 0.4957 rpy=3.14159 2.48154e-24 1.5708
- joint closing_BR_leg3_1 (1) (1)_1_frame: origin xyz=0.027272 -0.0419075 2.22045e-16 rpy=-3.0083e-16 2.4348e-15 -2.56468 -> xyz=0.027272 -0.0419075 1.63064e-16 rpy=-3.0083e-16 2.4348e-15 -2.56468
- joint closing_BR_leg3_1 (1) (1)_2_frame: origin xyz=0 -0.207 0 rpy=-3.14159 2.92432e-32 1.5708 -> xyz=-1.38778e-17 -0.207 0 rpy=-3.14159 2.92432e-32 1.5708
- joint closing_BR_leg3_1 (1) (1)_2_z_frame: origin xyz=2.77556e-17 -0.207 -0.1 rpy=-3.14159 2.92432e-32 1.5708 -> xyz=0 -0.207 -0.1 rpy=-3.14159 2.92432e-32 1.5708
- joint imu_link_frame: origin xyz=0.6663 -0.0247675 0.518956 rpy=3.30424e-16 8.36432e-16 -2.58163e-15 -> xyz=-0.0195 -0.015 0.0685 rpy=-2.48154e-24 -6.93889e-16 -2.22045e-16
- joint l: origin xyz=0.6808 0.0647675 0.432956 rpy=-1.5708 0.628319 -1.5708 -> xyz=-0.005 0.074535 -0.0175 rpy=-1.5708 0.628319 -1.5708
- joint pitch: origin xyz=1.21116e-17 -0.149706 0.0105 rpy=-1.5708 1.5708 0 -> xyz=-1.11022e-16 -0.149706 0.0105 rpy=-1.5708 1.5708 0
- joint yaw: origin xyz=1.11022e-16 0.0105 0.498956 rpy=1.5708 7.752e-16 -1.66569e-15 -> xyz=-0.6858 0.0202675 0.0485 rpy=1.5708 -7.55122e-16 4.71845e-16

Commit message: Automated update by GitHub Action

File: urdf/robot.urdf (robot description, URDF)
Before this commit: robot robot, 24 links, 23 joints
Links:
- removed link base_link_motor_holder
- removed link base_link_part_1_2
- removed link base_link_part_1_3
- removed link base_link_part_1_4
- removed link base_link_t_slot_frame
- removed link part_1_2
- added link hip_link, mass 1.06123; collision mesh filename=package://catbot_leg_description/meshes/motor_holder.stl; collision mesh filename=package://catbot_leg_description/meshes/part_1__3.stl
- link base_link_part_1: mass 0.0319952 -> 4.06535
- link part_1: geometry collision mesh filename=package://catbot_leg_description/meshes/part_1__2.stl; visual mesh filename=package://catbot_leg_description/meshes/part_1__2.stl
Joints:
- removed joint base_link_motor_holder_fixed
- removed joint base_link_part_1_2_fixed
- removed joint base_link_part_1_3_fixed
- removed joint base_link_part_1_4_fixed
- removed joint base_link_t_slot_frame_fixed
- joint BR_leg1_1 (1) (1): origin xyz=1.38778e-17 3.46945e-17 0.029 rpy=3.14159 1.11382e-16 -1.20167 -> xyz=0 0 0.029 rpy=3.14159 1.11382e-16 -1.20167
- joint BR_leg_cyl_0_1 (1) (1): origin xyz=-1.38778e-17 -0.166278 0 rpy=3.14159 3.7907e-32 1.13039e-17 -> xyz=-5.55112e-17 -0.166278 0 rpy=3.14159 3.7907e-32 1.13039e-17
- joint BR_leg_cyl_1_1 (1) (1): origin xyz=1.38778e-17 -0.207 0 rpy=-3.14159 -1.4511e-31 -6.07804e-18 -> xyz=2.77556e-17 -0.207 -1.11022e-16 rpy=-3.14159 -1.4511e-31 -6.07804e-18
- joint a: origin xyz=-0.005 -0.0545 -0.0175 rpy=1.5708 -1.25664 1.5708 -> xyz=0.6808 0.066 -0.0747675 rpy=-1.5708 -0.314159 -1.5708; parent base_link -> hip_link
- joint base_link_part_1_fixed: origin xyz=-0.0125 -0.0545 -0.0175 rpy=1.16838e-15 -1.91646e-16 1.5708 -> xyz=0 0 0 rpy=0 -0 1.5708
- joint closing_BR_leg3_1 (1) (1)_1_frame: origin xyz=0.027272 -0.0419075 1.63064e-16 rpy=-3.0083e-16 2.4348e-15 -2.56468 -> xyz=0.027272 -0.0419075 2.22045e-16 rpy=-3.0083e-16 2.4348e-15 -2.56468
- joint closing_BR_leg3_1 (1) (1)_2_frame: origin xyz=-1.38778e-17 -0.207 0 rpy=-3.14159 2.92432e-32 1.5708 -> xyz=-5.55112e-17 -0.207 0 rpy=-3.14159 2.92432e-32 1.5708
- joint closing_BR_leg3_1 (1) (1)_2_z_frame: origin xyz=0 -0.207 -0.1 rpy=-3.14159 2.92432e-32 1.5708 -> xyz=-5.55112e-17 -0.207 -0.1 rpy=-3.14159 2.92432e-32 1.5708
- joint imu_link_frame: origin xyz=-0.0195 -0.015 0.0685 rpy=-2.48154e-24 -6.93889e-16 -2.22045e-16 -> xyz=0.6663 -0.02 -0.0352675 rpy=1.5708 6.93889e-16 6.12323e-17; parent base_link -> hip_link
- joint l: origin xyz=-0.005 0.074535 -0.0175 rpy=-1.5708 0.628319 -1.5708 -> xyz=0.6808 0.066 0.0542675 rpy=1.5708 0.942478 1.5708; parent base_link -> hip_link
- joint pitch: child part_1_2 -> part_1; origin xyz=-1.11022e-16 -0.149706 0.0105 rpy=-1.5708 1.5708 0 -> xyz=-1.04083e-17 0 0.34925 rpy=3.14159 -0 1.5708; parent part_1 -> base_link
- joint yaw: child part_1 -> hip_link; origin xyz=-0.6858 0.0202675 0.0485 rpy=1.5708 -7.55122e-16 4.71845e-16 -> xyz=0.0105 -7.08145e-18 -0.149706 rpy=1.5708 7.55122e-16 1.5708; parent base_link -> part_1

Commit message: Automated update by GitHub Action

File: urdf/robot.urdf (robot description, URDF)
Before this commit: robot robot, 19 links, 18 joints
Links:
- removed link base_link_part_1
- link base_link: mass 1e-09 -> 4.06535; geometry collision mesh filename=package://catbot_leg_description/meshes/part_1.stl; visual mesh filename=package://catbot_leg_description/meshes/part_1.stl
Joints:
- removed joint base_link_part_1_fixed
- joint pitch: child part_1 -> hip_link; origin xyz=-1.04083e-17 0 0.34925 rpy=3.14159 -0 1.5708 -> xyz=0.0105 -7.08145e-18 -0.149706 rpy=1.5708 7.55122e-16 1.5708; parent base_link -> part_1
- joint yaw: child hip_link -> part_1; limit lower=-3.141592653589793 upper=3.141592653589793 effort=10 velocity=10 -> effort=10 velocity=10; origin xyz=0.0105 -7.08145e-18 -0.149706 rpy=1.5708 7.55122e-16 1.5708 -> xyz=-1.04083e-17 0 0.34925 rpy=3.14159 -0 1.5708; parent part_1 -> base_link; type revolute -> continuous

Commit message: Automated update by GitHub Action

File: urdf/robot.urdf (robot description, URDF)
Before this commit: robot robot, 18 links, 17 joints
Joints:
- joint BR_leg1_1 (1) (1): limit lower=-3.141592653589793 upper=3.141592653589793 effort=10 velocity=10 -> lower=-0.119564 upper=2.0621 effort=10 velocity=10; origin xyz=0 0 0.029 rpy=3.14159 1.11382e-16 -1.20167 -> xyz=-5.55112e-17 -1.11022e-16 0.029 rpy=-3.14159 6.91027e-16 -1.20167
- joint BR_leg2_1 (1) (1): limit lower=-3.141592653589793 upper=3.141592653589793 effort=10 velocity=10 -> lower=-0.135581 upper=2.22061 effort=10 velocity=10; origin xyz=0.0292942 0.0403199 0.029 rpy=3.14159 1.98827e-15 -1.20023 -> xyz=0.0292942 0.0403199 0.029 rpy=3.14159 1.46668e-15 -1.20023
- joint BR_leg_cyl_0_1 (1) (1): origin xyz=-5.55112e-17 -0.166278 0 rpy=3.14159 3.7907e-32 1.13039e-17 -> xyz=2.77556e-17 -0.166278 -1.11022e-16 rpy=-3.14159 -6.74381e-32 -2.54852e-17
- joint BR_leg_cyl_1_1 (1) (1): limit lower=-3.141592653589793 upper=3.141592653589793 effort=10 velocity=10 -> lower=-0.140581 upper=2.12835 effort=10 velocity=10; origin xyz=2.77556e-17 -0.207 -1.11022e-16 rpy=-3.14159 -1.4511e-31 -6.07804e-18 -> xyz=5.55112e-17 -0.207 -1.11022e-16 rpy=3.14159 -4.88264e-31 5.70903e-17
- joint a: limit lower=-3.141592653589793 upper=3.141592653589793 effort=10 velocity=10 -> lower=-2.70526 upper=0.261799 effort=10 velocity=10
- joint closing_BR_leg0_1 (1) (1)_1_frame: origin xyz=0.0748567 -0.0443336 -0.001 rpy=2.31825e-17 3.12039e-18 -2.1055 -> xyz=0.0748567 -0.0443336 -0.001 rpy=9.11366e-15 -7.23279e-15 -2.1055
- joint closing_BR_leg0_1 (1) (1)_1_z_frame: origin xyz=0.0748567 -0.0443336 0.099 rpy=2.31825e-17 3.12039e-18 -2.1055 -> xyz=0.0748567 -0.0443336 0.099 rpy=9.11366e-15 -7.23279e-15 -2.1055
- joint closing_BR_leg0_1 (1) (1)_2_frame: origin xyz=-0.0588116 -0.0191091 0.028 rpy=-2.17485e-14 1.40298e-14 0.314159 -> xyz=-0.0588116 -0.0191091 0.028 rpy=9.7098e-16 -2.75934e-16 0.314159
- joint closing_BR_leg0_1 (1) (1)_2_z_frame: origin xyz=-0.0588116 -0.0191091 0.128 rpy=-2.17485e-14 1.40298e-14 0.314159 -> xyz=-0.0588116 -0.0191091 0.128 rpy=9.7098e-16 -2.75934e-16 0.314159
- joint closing_BR_leg3_1 (1) (1)_1_frame: origin xyz=0.027272 -0.0419075 2.22045e-16 rpy=-3.0083e-16 2.4348e-15 -2.56468 -> xyz=0.027272 -0.0419075 -6.66134e-16 rpy=-1.22687e-14 -2.27337e-15 -2.56468
- joint closing_BR_leg3_1 (1) (1)_1_z_frame: origin xyz=0.027272 -0.0419075 0.1 rpy=-3.0083e-16 2.4348e-15 -2.56468 -> xyz=0.027272 -0.0419075 0.1 rpy=-1.22687e-14 -2.27337e-15 -2.56468
- joint closing_BR_leg3_1 (1) (1)_2_frame: origin xyz=-5.55112e-17 -0.207 0 rpy=-3.14159 2.92432e-32 1.5708 -> xyz=2.77556e-17 -0.207 0 rpy=3.14159 -3.96308e-31 1.5708
- joint closing_BR_leg3_1 (1) (1)_2_z_frame: origin xyz=-5.55112e-17 -0.207 -0.1 rpy=-3.14159 2.92432e-32 1.5708 -> xyz=2.77556e-17 -0.207 -0.1 rpy=3.14159 -3.96308e-31 1.5708
- joint l: limit lower=-3.141592653589793 upper=3.141592653589793 effort=10 velocity=10 -> lower=-1.0472 upper=2.18166 effort=10 velocity=10
- joint pitch: origin xyz=0.0105 -7.08145e-18 -0.149706 rpy=1.5708 7.55122e-16 1.5708 -> xyz=0.0105 1.54859e-16 -0.149706 rpy=1.5708 -1.31896e-14 1.5708
- joint yaw: origin xyz=-1.04083e-17 0 0.34925 rpy=3.14159 -0 1.5708 -> xyz=-1.73472e-18 0 0.34925 rpy=-3.14159 1.21905e-17 1.5708

Commit message: Automated update by GitHub Action

File: urdf/robot.urdf (robot description, URDF)
Before this commit: robot robot, 18 links, 17 joints
Links:
- link hip_link: mass 1.06123 -> 1.05519
Joints:
- joint BR_leg1_1 (1) (1): origin xyz=-5.55112e-17 -1.11022e-16 0.029 rpy=-3.14159 6.91027e-16 -1.20167 -> xyz=-1.11022e-16 -1.66533e-16 0.029 rpy=-3.14159 5.73317e-16 -1.20167
- joint BR_leg2_1 (1) (1): origin xyz=0.0292942 0.0403199 0.029 rpy=3.14159 1.46668e-15 -1.20023 -> xyz=0.0292942 0.0403199 0.029 rpy=-3.14159 1.34653e-15 -1.20023
- joint l: limit lower=-1.0472 upper=2.18166 effort=10 velocity=10 -> lower=-0.174533 upper=2.18166 effort=10 velocity=10
